File: Kicad/outputs.sch (KiCad schematic (older format))
At the start: 0 parts

Commit message: added CV output buffers
Parts:
- added C? (x2): 22pF, symbol Device:C_Small
- added D? (x2): LED, symbol Device:LED
- added J?: CV_OUT_1, Connector_Audio:Jack_3.5mm_QingPu_WQP-PJ398SM_Vertical_CircularHoles, symbol Connector:AudioJack2_SwitchT
- added J?: TRIG_OUT_1, Connector_Audio:Jack_3.5mm_QingPu_WQP-PJ398SM_Vertical_CircularHoles, symbol Connector:AudioJack2_SwitchT
- added J?: TRIG_OUT_2, Connector_Audio:Jack_3.5mm_QingPu_WQP-PJ398SM_Vertical_CircularHoles, symbol Connector:AudioJack2_SwitchT
- added J?: CV_OUT_2, Connector_Audio:Jack_3.5mm_QingPu_WQP-PJ398SM_Vertical_CircularHoles, symbol Connector:AudioJack2_SwitchT
- added Q? (x2): 2N3904, Package_TO_SOT_THT:TO-92_Inline, symbol Transistor_BJT:2N3904
- added R, R?: 1k, symbol Device:R_Small
- added R? (x4): 10k, symbol Device:R_Small
- added R? (x2): 1k, symbol Device:R
- added R? (x2): R1k, symbol Device:R
- added R? (x2): 120, symbol Device:R
- added R? (x2): 1k8, symbol Device:R
- added U? (x2): TL072, symbol Amplifier_Operational:TL072
Connections:
- new net: C?.1, R.2, U?.1
- new net: C?.2, R?.2, R?.2, U?.2 (-)
- new net: C?.2, R?.2, R?.2, U?.6 (-)
- new net: C?.1, R?.2, U?.7
- new net: J?.T, R.1, R?.1
- new net: D?.2 (A), R?.2 (x2)
- new net: Q?.2 (B), R?.1 (x2)
- new net: J?.T, R?.1 (x2)
- new net: Q?.3 (C), R?.1, R?.2 (x2)
- new net: J?.T, R?.1, R?.1
- new net +5V: R?.1, R?.1, R?.2, R?.2
- new net DAC_1: U?.3 (+)
- new net DAC_2: U?.5 (+)
- new net GND: J?.S, J?.S, J?.S, J?.S, Q?.1 (E), Q?.1 (E), R?.1, R?.1
- new net MCU_TRIG_OUT_1: D?.1 (K), R?.2
- new net MCU_TRIG_OUT_2: D?.1 (K), R?.2
Other:
- note added: "CV outputs"
- note added: "Trigger/Gate outputs"
