File: Kicad/inputs_outputs.sch (KiCad schematic (older format))
At the start: 40 parts

Commit message: completing schematics and starting to correct errors
Parts:
- gave numbers to parts that had none: 38
- renumbered R to R21

Commit message: correcting some connections
Connections:
- no-connect marks 0 -> 6
Changed lines of the file:
@@
 Text Notes 720  1260 0    50   ~ 0
 Triggers/Gates inputs
+NoConn ~ 10070 1170
+NoConn ~ 10070 2960
+NoConn ~ 7110 3420
+NoConn ~ 7060 5270
+NoConn ~ 1580 3910
+NoConn ~ 1580 2220
 $EndSCHEMATC

Commit message: updated power section with switching regulator
Other:
- moved on the sheet: D3, D4, D5, D6, J1, J2, J3, J4, Q1, Q2, Q3, Q4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
